File: lm27762/lm27762.kicad_sch (KiCad schematic)
At the start: 18 parts, among them J1 Conn_01x04

Commit message: updated design files to RevA
Parts:
- removed D1: LED, LED_SMD:LED_0402_1005Metric_Pad0.77x0.64mm_HandSolder, symbol Device:LED
- added C1: 10u, Capacitor_SMD:C_0603_1608Metric_Pad1.08x0.95mm_HandSolder, symbol Device:C
- C2: renamed from CIN1; LCSC (none) -> C52923; MPN (none) -> CL05A105KA5NQNC
- CF1: renamed from C1; LCSC (none) -> C14445; MPN (none) -> CL05A105KP5NNNC
- CO1, CO2: value 1u -> 2.2u; footprint Capacitor_SMD:C_0402_1005Metric_Pad0.74x0.62mm_HandSolder -> Capacitor_SMD:C_0603_1608Metric_Pad1.08x0.95mm_HandSolder; LCSC (none) -> C1607; MPN (none) -> CL10A225KP8NNNC
- CP1: renamed from CCP1; value 1u -> 4.7u; footprint Capacitor_SMD:C_0402_1005Metric_Pad0.74x0.62mm_HandSolder -> Capacitor_SMD:C_0603_1608Metric_Pad1.08x0.95mm_HandSolder; LCSC (none) -> C1705; MPN (none) -> CL10A475KP8NNNC
- R1, R3: value ~ -> 680k; footprint Resistor_SMD:R_0402_1005Metric_Pad0.72x0.64mm_HandSolder -> Resistor_SMD:R_0603_1608Metric_Pad0.98x0.95mm_HandSolder; LCSC (none) -> C137690; MPN (none) -> RC0603FR-07680KL
- R2, R4: value ~ -> 220k; footprint Resistor_SMD:R_0402_1005Metric_Pad0.72x0.64mm_HandSolder -> Resistor_SMD:R_0603_1608Metric_Pad0.98x0.95mm_HandSolder; LCSC (none) -> C123420; MPN (none) -> RC0603FR-07220KL
- RP1: LCSC (none) -> C191123; MPN (none) -> ERJ2RKF1002X
- TP2, TP3, TP4, TP6, TP7: footprint TestPoint:TestPoint_Pad_D1.0mm -> TinyTestPoints:0_5mm
- U1: value ~ -> LM27762DSSR; LCSC (none) -> C473398; MPN (none) -> LM27762DSSR
Connections:
- net GND: now also C1.2
- net VIN: now also RP1.2, C1.1
